File: Hardware/Tilt-A-Whirl_RPI-1031.brd (EAGLE design)
At the start: 10.2 x 10.2 mm, 11 parts, among them U1 RPI-1031

Commit message: Updating board/schematic from review
Parts:
- moved U$1 0.90 mm to (7.62, 8.26), turned to 270 degrees
- moved U1 0.63 mm to (7.62, 4.45)
Routing:
- net AN: track 3.07 -> 2.25 mm
Changed lines of the file:
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@@
 </class>
 </classes>
-<designrules name="SparkFun">
+<designrules name="SparkFun *">
 <description language="en">&lt;b&gt;EAGLE Design Rules&lt;/b&gt;
 &lt;p&gt;
@@
 <param name="dpGapFactor" value="2.5"/>
 <param name="checkGrid" value="0"/>
-<param name="checkAngle" value="0"/>
+<param name="checkAngle" value="1"/>
 <param name="checkFont" value="1"/>
 <param name="checkRestrict" value="1"/>
@@
 </autorouter>
 <elements>
-<element name="U1" library="Local Lirary" package="RPI-1031" value="RPI-1031" x="7.62" y="5.08" rot="R90"/>
+<element name="U1" library="Local Lirary" package="RPI-1031" value="RPI-1031" x="7.62" y="4.445" rot="R90"/>
 <element name="JP4" library="SparkFun" package="SFE-LOGO-FLAME" value="LOGO-SFESK" x="2.921" y="9.525" rot="R270"/>
 <element name="JP1" library="SparkFun" package="1X04" value="" x="1.27" y="1.27" rot="R90"/>
@@
 <attribute name="VALUE" value="240" x="7.62" y="1.27" size="1.778" layer="27" rot="R180" display="off"/>
 </element>
-<element name="U$1" library="SparkFun" package="OSHW-LOGO-S" value="OSHW-LOGOS" x="8.255" y="8.89" rot="R180"/>
+<element name="U$1" library="SparkFun" package="OSHW-LOGO-S" value="OSHW-LOGOS" x="7.62" y="8.255" rot="R270"/>
 <element name="JP2" library="abes" package="FIDUCIAL-1X2.5" value="FIDUCIAL1X2.5" x="9.4742" y="9.5504"/>
 <element name="JP3" library="abes" package="FIDUCIAL-1X2.5" value="FIDUCIAL1X2.5" x="3.2258" y="0.635"/>
@@
 <contactref element="R2" pad="1"/>
 <contactref element="R1" pad="1"/>
-<via x="7.62" y="8.89" extent="1-16" drill="0.508"/>
+<via x="5.842" y="9.271" extent="1-16" drill="0.508"/>
 <via x="5.08" y="1.27" extent="1-16" drill="0.508"/>
 <polygon width="0.254" layer="1" isolate="0.3048">
@@
 <wire x1="3.81" y1="4.865" x2="3.595" y2="4.865" width="0.254" layer="1"/>
 <wire x1="3.595" y1="4.865" x2="2.54" y2="3.81" width="0.254" layer="1"/>
-<wire x1="6.175" y1="6.3" x2="5.665" y2="6.3" width="0.254" layer="1"/>
-<wire x1="3.81" y1="4.865" x2="4.23" y2="4.865" width="0.254" layer="1"/>
-<wire x1="4.23" y1="4.865" x2="5.665" y2="6.3" width="0.254" layer="1"/>
+<wire x1="6.175" y1="5.665" x2="5.03" y2="5.665" width="0.254" layer="1"/>
+<wire x1="5.03" y1="5.665" x2="4.445" y2="5.08" width="0.254" layer="1"/>
+<wire x1="4.445" y1="5.08" x2="4.025" y2="5.08" width="0.254" layer="1"/>
+<wire x1="4.025" y1="5.08" x2="3.81" y2="4.865" width="0.254" layer="1"/>
 </signal>
 <signal name="AN">
 <contactref element="U1" pad="6"/>
 <contactref element="R3" pad="1"/>
-<wire x1="8.975" y1="3.95" x2="8.975" y2="3.26" width="0.254" layer="1"/>
-<wire x1="8.975" y1="3.26" x2="8.255" y2="2.54" width="0.254" layer="1"/>
-<wire x1="8.255" y1="2.54" x2="8.255" y2="1.485" width="0.254" layer="1"/>
-<wire x1="8.255" y1="1.485" x2="8.47" y2="1.27" width="0.254" layer="1"/>
+<wire x1="8.975" y1="3.315" x2="8.975" y2="2.498" width="0.254" layer="1"/>
+<wire x1="8.975" y1="2.498" x2="8.509" y2="2.032" width="0.254" layer="1"/>
+<wire x1="8.509" y1="2.032" x2="8.509" y2="1.309" width="0.254" layer="1"/>
+<wire x1="8.509" y1="1.309" x2="8.47" y2="1.27" width="0.254" layer="1"/>
 </signal>
 <signal name="S2">
@@
 <contactref element="U1" pad="4"/>
 <contactref element="R2" pad="2"/>
-<wire x1="6.175" y1="3.95" x2="5.22" y2="3.95" width="0.254" layer="1"/>
-<wire x1="3.81" y1="3.39" x2="4.66" y2="3.39" width="0.254" layer="1"/>
-<wire x1="4.66" y1="3.39" x2="5.22" y2="3.95" width="0.254" layer="1"/>
 <wire x1="3.81" y1="3.39" x2="3.39" y2="3.39" width="0.254" layer="1"/>
 <wire x1="3.39" y1="3.39" x2="1.27" y2="1.27" width="0.254" layer="1"/>
+<wire x1="3.81" y1="3.39" x2="6.1" y2="3.39" width="0.254" layer="1"/>
+<wire x1="6.1" y1="3.39" x2="6.175" y2="3.315" width="0.254" layer="1"/>
 </signal>
 <signal name="5V">
@@
 <contactref element="U1" pad="5"/>
 <contactref element="U1" pad="2"/>
-<wire x1="7.575" y1="3.95" x2="7.575" y2="6.3" width="0.254" layer="1"/>
-<wire x1="7.575" y1="3.95" x2="7.575" y2="3.13" width="0.254" layer="1"/>
-<wire x1="7.575" y1="3.13" x2="6.985" y2="2.54" width="0.254" layer="1"/>
-<wire x1="6.985" y1="2.54" x2="6.985" y2="1.485" width="0.254" layer="1"/>
-<wire x1="6.985" y1="1.485" x2="6.77" y2="1.27" width="0.254" layer="1"/>
-<wire x1="7.575" y1="6.3" x2="7.575" y2="7.665" width="0.254" layer="1"/>
+<wire x1="7.575" y1="3.315" x2="7.575" y2="5.665" width="0.254" layer="1"/>
+<wire x1="7.575" y1="5.665" x2="7.575" y2="7.665" width="0.254" layer="1"/>
 <wire x1="7.575" y1="7.665" x2="6.985" y2="8.255" width="0.254" layer="1"/>
 <wire x1="6.985" y1="8.255" x2="1.905" y2="8.255" width="0.254" layer="1"/>
 <wire x1="1.905" y1="8.255" x2="1.27" y2="8.89" width="0.254" layer="1"/>
+<wire x1="7.575" y1="3.315" x2="7.575" y2="2.495" width="0.254" layer="1"/>
+<wire x1="7.575" y1="2.495" x2="6.985" y2="1.905" width="0.254" layer="1"/>
+<wire x1="6.985" y1="1.905" x2="6.985" y2="1.485" width="0.254" layer="1"/>
+<wire x1="6.985" y1="1.485" x2="6.77" y2="1.27" width="0.254" layer="1"/>
 </signal>
 </signals>
